File: hardware/Electrical schematic/schematic.kicad_sch (KiCad schematic)
At the start: 12 parts, among them M1 Motor_DC, M2 Motor_DC, SW1 SW_Push, SW2 SW_DPST, U1 NUCLEO-H533RE, U2 IR, U3 IR, U4 Sharp, U5 Sharp, U6 Sharp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

Commit message: fix: updated electrical schematic based on review
Parts:
- removed SW2: SW_DPST, symbol Switch:SW_DPST_x2
- added SW3: SW_SPST, symbol Switch:SW_SPST
Connections:
- net at U1. (VIN), U7. (OUT4): now also SW3.1 (A)
- net at BT1.1 (+): now also SW3.2 (B)
- new net: BT1.2 (-), U1. (VIN), U2. (OUT), U3. (OUT), U4. (OUT), U5. (OUT), U6. (OUT), U7. (OUT4)
- new net: U1. (VIN), U4. (OUT), U5. (OUT), U6. (OUT)
- new net: SW1.1, U1. (VIN), U2. (OUT), U3. (OUT)
Other:
- company: (none) -> CybAiR
- title: minisumo -> degradoinator
